Commit message: 2024 11 12: Able to show robot and room properly in gazebo

File: src/robot_description/urdf/MicroROS.urdf (robot description, URDF)
Before this commit: robot micro4.0, 9 links, 8 joints
Links:
- link base_link: geometry collision mesh filename=file:///home/kunama/PLCT/NAV2/nav2_sim/src/robot_descriptio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; visual mesh filename=file:///home/kunama/PLCT/NAV2/nav2_sim/src/robot_descriptio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
- link imu_Link: geometry collision mesh filename=file:///home/kunama/PLCT/NAV2/nav2_sim/src/robot_descriptio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; visual mesh filename=file:///home/kunama/PLCT/NAV2/nav2_sim/src/robot_descriptio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
- link jq1_Link: geometry collision mesh filename=file:///home/kunama/PLCT/NAV2/nav2_sim/src/robot_descriptio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; visual mesh filename=file:///home/kunama/PLCT/NAV2/nav2_sim/src/robot_descriptio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
- link jq2_Link: geometry collision mesh filename=file:///home/kunama/PLCT/NAV2/nav2_sim/src/robot_descriptio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; visual mesh filename=file:///home/kunama/PLCT/NAV2/nav2_sim/src/robot_descriptio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
- link radar_Link: geometry collision mesh filename=file:///home/kunama/PLCT/NAV2/nav2_sim/src/robot_descriptio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; visual mesh filename=file:///home/kunama/PLCT/NAV2/nav2_sim/src/robot_descriptio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
- link yh_Link: geometry collision mesh filename=file:///home/kunama/PLCT/NAV2/nav2_sim/src/robot_descriptio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; visual mesh filename=file:///home/kunama/PLCT/NAV2/nav2_sim/src/robot_descriptio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
- link yq_Link: geometry collision mesh filename=file:///home/kunama/PLCT/NAV2/nav2_sim/src/robot_descriptio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; visual mesh filename=file:///home/kunama/PLCT/NAV2/nav2_sim/src/robot_descriptio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
- link zh_Link: geometry collision mesh filename=file:///home/kunama/PLCT/NAV2/nav2_sim/src/robot_descriptio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; visual mesh filename=file:///home/kunama/PLCT/NAV2/nav2_sim/src/robot_descriptio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
- link zq_Link: geometry collision mesh filename=file:///home/kunama/PLCT/NAV2/nav2_sim/src/robot_descriptio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; visual mesh filename=file:///home/kunama/PLCT/NAV2/nav2_sim/src/robot_descriptio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

Commit message: adding pakcge robot slam

File: src/robot_description/urdf/MicroROS.urdf (robot description, URDF)
Before this commit: robot micro4.0, 9 links, 8 joints
Joints:
- joint zh_Joint: axis 0 1 0 -> 0 -1 0
- joint zq_Joint: axis 0 1 0 -> 0 -1 0

Commit message: able to drive in diff mode with keyboard

File: src/robot_description/urdf/MicroROS.urdf (robot description, URDF)
Before this commit: robot micro4.0, 9 links, 8 joints
Links:
- link base_link: geometry collision mesh filename=file:///mnt/nvme1n1p6/PLCT/NAV2/nav2_sim/src/robot_descript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; visual mesh filename=file:///mnt/nvme1n1p6/PLCT/NAV2/nav2_sim/src/robot_descript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
- link imu_Link: geometry collision mesh filename=file:///mnt/nvme1n1p6/PLCT/NAV2/nav2_sim/src/robot_descript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; visual mesh filename=file:///mnt/nvme1n1p6/PLCT/NAV2/nav2_sim/src/robot_descript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
- link jq1_Link: geometry collision mesh filename=file:///mnt/nvme1n1p6/PLCT/NAV2/nav2_sim/src/robot_descript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; visual mesh filename=file:///mnt/nvme1n1p6/PLCT/NAV2/nav2_sim/src/robot_descript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
- link jq2_Link: geometry collision mesh filename=file:///mnt/nvme1n1p6/PLCT/NAV2/nav2_sim/src/robot_descript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; visual mesh filename=file:///mnt/nvme1n1p6/PLCT/NAV2/nav2_sim/src/robot_descript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
- link radar_Link: geometry collision mesh filename=file:///mnt/nvme1n1p6/PLCT/NAV2/nav2_sim/src/robot_descript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; visual mesh filename=file:///mnt/nvme1n1p6/PLCT/NAV2/nav2_sim/src/robot_descript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
- link yh_Link: geometry collision mesh filename=file:///mnt/nvme1n1p6/PLCT/NAV2/nav2_sim/src/robot_descript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; visual mesh filename=file:///mnt/nvme1n1p6/PLCT/NAV2/nav2_sim/src/robot_descript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
- link yq_Link: geometry collision mesh filename=file:///mnt/nvme1n1p6/PLCT/NAV2/nav2_sim/src/robot_descript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; visual mesh filename=file:///mnt/nvme1n1p6/PLCT/NAV2/nav2_sim/src/robot_descript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
- link zh_Link: geometry collision mesh filename=file:///mnt/nvme1n1p6/PLCT/NAV2/nav2_sim/src/robot_descript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; visual mesh filename=file:///mnt/nvme1n1p6/PLCT/NAV2/nav2_sim/src/robot_descript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
- link zq_Link: geometry collision mesh filename=file:///mnt/nvme1n1p6/PLCT/NAV2/nav2_sim/src/robot_descript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; visual mesh filename=file:///mnt/nvme1n1p6/PLCT/NAV2/nav2_sim/src/robot_descript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

Commit message: modified path

File: src/robot_description/urdf/MicroROS.urdf (robot description, URDF)
Before this commit: robot micro4.0, 9 links, 8 joints
Links:
- link base_link: geometry collision mesh filename=package://robot_description/meshes/MicroROS/base_link.STL; visual mesh filename=package://robot_description/meshes/MicroROS/base_link.STL
- link imu_Link: geometry collision mesh filename=package://robot_description/meshes/MicroROS/imu_Link.STL; visual mesh filename=package://robot_description/meshes/MicroROS/imu_Link.STL
- link jq1_Link: geometry collision mesh filename=package://robot_description/meshes/MicroROS/jq1_Link.STL; visual mesh filename=package://robot_description/meshes/MicroROS/jq1_Link.STL
- link jq2_Link: geometry collision mesh filename=package://robot_description/meshes/MicroROS/jq2_Link.STL; visual mesh filename=package://robot_description/meshes/MicroROS/jq2_Link.STL
- link radar_Link: geometry collision mesh filename=package://robot_description/meshes/MicroROS/radar_Link.STL; visual mesh filename=package://robot_description/meshes/MicroROS/radar_Link.STL
- link yh_Link: geometry collision mesh filename=package://robot_description/meshes/MicroROS/yh_Link.STL; visual mesh filename=package://robot_description/meshes/MicroROS/yh_Link.STL
- link yq_Link: geometry collision mesh filename=package://robot_description/meshes/MicroROS/yq_Link.STL; visual mesh filename=package://robot_description/meshes/MicroROS/yq_Link.STL
- link zh_Link: geometry collision mesh filename=package://robot_description/meshes/MicroROS/zh_Link.STL; visual mesh filename=package://robot_description/meshes/MicroROS/zh_Link.STL
- link zq_Link: geometry collision mesh filename=package://robot_description/meshes/MicroROS/zq_Link.STL; visual mesh filename=package://robot_description/meshes/MicroROS/zq_Link.STL
