Commit message: update urdf

File: src/robot_description/urdf/A2_W.urdf (robot description, URDF)
Before this commit: robot raise_a2_w_t3, 43 links, 42 joints
Joints:
- joint idx10_waist_joint: type revolute -> fixed

Commit message: upload the test src of gazebo-nav2 simulation src in openeuler

File: src/robot_description/urdf/A2_W.urdf (robot description, URDF)
Before this commit: robot raise_a2_w_t3, 43 links, 42 joints
Links:
- link arm_base_link: geometry collision box size=0.16 0.27200043 0.12292724999999999; visual mesh filename=package:///robot_description/meshes/A2_W/arm_base_link.STL
- link base_link: geometry collision box size=0.3759756 0.38513064 1.2152664999999998; collision box size=0.44176495 0.41260087 0.07947397
- link body_link1: geometry collision box size=0.190643 0.297199 0.184147; visual mesh filename=package:///robot_description/meshes/A2_W/body_link1.STL scale=1.0 1.0 1.0
- link body_link2: geometry collision box size=0.20786262 0.51781845 0.18883516; visual mesh filename=package:///robot_description/meshes/A2_W/body_link2.STL scale=1.0 1.0 1.0
- link head_link: geometry collision box size=0.1024513691663742 0.1386224739253521 0.12076015025377274; visual mesh filename=package:///robot_description/meshes/A2_W/head_link.STL scale=1.0 1.0 1.0
- link left_arm_link01: geometry collision cylinder length=0.14799022674560547 radius=0.0522; visual mesh filename=package:///robot_description/meshes/A2_W/l1.STL
- link left_arm_link02: geometry collision box size=0.10358428955078125 0.17078391090035439 0.12926186621189117; visual mesh filename=package:///robot_description/meshes/A2_W/l2.STL
- link left_arm_link03: geometry collision box size=0.10300003 0.1029582 0.21228018000000004; visual mesh filename=package:///robot_description/meshes/A2_W/l3.STL
- link left_arm_link04: geometry collision box size=0.09023327 0.12190476 0.10766125; collision cylinder length=.10766125 radius=0.048
- link left_arm_link05: geometry collision box size=0.08318585157394409 0.0841069221496582 0.16509421914815903; visual mesh filename=package:///robot_description/meshes/A2_W/l5.STL
- link left_arm_link06: geometry collision box size=0.08100000023841858 0.19017678871750832 0.08721351623535156; visual mesh filename=package:///robot_description/meshes/A2_W/l6.STL
- link left_arm_link07_transition: geometry collision cylinder length=0.0495000034570694 radius=0.040500002409446435; visual mesh filename=package:///robot_description/meshes/A2_W/l7.STL
- link left_finger_base: geometry collision box size=0.06199646 0.06209 0.06850052; collision box size=0.0987854 0.10564122 0.13784218
- link left_finger_left: geometry collision box size=0.04345703 0.02092956 0.107421875; visual mesh filename=package:///robot_description/meshes/A2_W/finger.STL scale=0.001 0.001 0.001
- link left_finger_right: geometry collision box size=0.04345703 0.02092956 0.107421875; visual mesh filename=package:///robot_description/meshes/A2_W/finger.STL scale=0.001 0.001 0.001
- link right_arm_link01: geometry collision cylinder length=0.14799022674560547 radius=0.0522; visual mesh filename=package:///robot_description/meshes/A2_W/r1.STL
- link right_arm_link02: geometry collision box size=0.10358428955078125 0.17078391090035439 0.12926186621189117; visual mesh filename=package:///robot_description/meshes/A2_W/r2.STL
- link right_arm_link03: geometry collision box size=0.10300003 0.1029582 0.21228018000000004; visual mesh filename=package:///robot_description/meshes/A2_W/r3.STL
- link right_arm_link04: geometry collision box size=0.09023327 0.12190476 0.10766125; collision cylinder length=0.10766125 radius=0.048
- link right_arm_link05: geometry collision box size=0.08318585157394409 0.0841069221496582 0.16509421914815903; visual mesh filename=package:///robot_description/meshes/A2_W/r5.STL
- link right_arm_link06: geometry collision box size=0.08100000023841858 0.19017678871750832 0.08721351623535156; visual mesh filename=package:///robot_description/meshes/A2_W/r6.STL
- link right_arm_link07_transition: geometry collision cylinder length=0.0495000034570694 radius=0.040500002385802265; visual mesh filename=package:///robot_description/meshes/A2_W/r7.STL
- link right_finger_base: geometry collision box size=0.06199646 0.06209 0.06850052; collision box size=0.0987854 0.10564122 0.13784218
- link right_finger_left: geometry collision box size=0.04345703 0.02092956 0.107421875; visual mesh filename=package:///robot_description/meshes/A2_W/finger.STL scale=0.001 0.001 0.001
- link right_finger_right: geometry collision box size=0.04345703 0.02092956 0.107421875; visual mesh filename=package:///robot_description/meshes/A2_W/finger.STL scale=0.001 0.001 0.001
- link wheel_1: geometry collision mesh filename=package:///robot_description/meshes/A2_W/wheel_1.STL scale=1.0 1.0 1.0; visual mesh filename=package:///robot_description/meshes/A2_W/wheel_1.STL scale=1.0 1.0 1.0
- link wheel_1_yaw: geometry visual mesh filename=package:///robot_description/meshes/A2_W/wheel_1_yaw.STL scale=1.0 1.0 1.0
- link wheel_2: geometry collision mesh filename=package:///robot_description/meshes/A2_W/wheel_2.STL scale=1.0 1.0 1.0; visual mesh filename=package:///robot_description/meshes/A2_W/wheel_2.STL scale=1.0 1.0 1.0
- link wheel_2_yaw: geometry visual mesh filename=package:///robot_description/meshes/A2_W/wheel_2_yaw.STL scale=1.0 1.0 1.0
- link wheel_3: geometry collision mesh filename=package:///robot_description/meshes/A2_W/wheel_3.STL scale=1.0 1.0 1.0; visual mesh filename=package:///robot_description/meshes/A2_W/wheel_3.STL scale=1.0 1.0 1.0
- link wheel_3_yaw: geometry visual mesh filename=package:///robot_description/meshes/A2_W/wheel_3_yaw.STL scale=1.0 1.0 1.0
- link wheel_4: geometry collision mesh filename=package:///robot_description/meshes/A2_W/wheel_4.STL scale=1.0 1.0 1.0; visual mesh filename=package:///robot_description/meshes/A2_W/wheel_4.STL scale=1.0 1.0 1.0
- link wheel_4_yaw: geometry visual mesh filename=package:///robot_description/meshes/A2_W/wheel_4_yaw.STL scale=1.0 1.0 1.0

File: src/robot_description/urdf/MicroROS.urdf (robot description, URDF)
Before this commit: robot micro4.0, 9 links, 8 joints
Links:
- link base_link: geometry collision mesh filename=file:///mnt/nvme1n1p6/PLCT/NAV2/nav2_sim/src/robot_descript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; visual mesh filename=file:///mnt/nvme1n1p6/PLCT/NAV2/nav2_sim/src/robot_descript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
- link imu_Link: geometry collision mesh filename=file:///mnt/nvme1n1p6/PLCT/NAV2/nav2_sim/src/robot_descript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; visual mesh filename=file:///mnt/nvme1n1p6/PLCT/NAV2/nav2_sim/src/robot_descript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
- link jq1_Link: geometry collision mesh filename=file:///mnt/nvme1n1p6/PLCT/NAV2/nav2_sim/src/robot_descript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; visual mesh filename=file:///mnt/nvme1n1p6/PLCT/NAV2/nav2_sim/src/robot_descript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
- link jq2_Link: geometry collision mesh filename=file:///mnt/nvme1n1p6/PLCT/NAV2/nav2_sim/src/robot_descript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; visual mesh filename=file:///mnt/nvme1n1p6/PLCT/NAV2/nav2_sim/src/robot_descript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
- link radar_Link: geometry collision mesh filename=file:///mnt/nvme1n1p6/PLCT/NAV2/nav2_sim/src/robot_descript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; visual mesh filename=file:///mnt/nvme1n1p6/PLCT/NAV2/nav2_sim/src/robot_descript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
- link yh_Link: geometry collision mesh filename=file:///mnt/nvme1n1p6/PLCT/NAV2/nav2_sim/src/robot_descript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; visual mesh filename=file:///mnt/nvme1n1p6/PLCT/NAV2/nav2_sim/src/robot_descript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
- link yq_Link: geometry collision mesh filename=file:///mnt/nvme1n1p6/PLCT/NAV2/nav2_sim/src/robot_descript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; visual mesh filename=file:///mnt/nvme1n1p6/PLCT/NAV2/nav2_sim/src/robot_descript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
- link zh_Link: geometry collision mesh filename=file:///mnt/nvme1n1p6/PLCT/NAV2/nav2_sim/src/robot_descript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; visual mesh filename=file:///mnt/nvme1n1p6/PLCT/NAV2/nav2_sim/src/robot_descript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
- link zq_Link: geometry collision mesh filename=file:///mnt/nvme1n1p6/PLCT/NAV2/nav2_sim/src/robot_descript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; visual mesh filename=file:///mnt/nvme1n1p6/PLCT/NAV2/nav2_sim/src/robot_descript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
